File: ROCSAR_Hardware/Interface_PCB/Interface_PCB.kicad_pcb (KiCad board)
At the start: 2 copper layers, 7 parts, among them J1 Remove Before Flight, U1 TEN 60-2422N

Commit message: PCB Update
Parts:
- removed C1: 0.1uF, Capacitor_SMD:C_1206_3216Metric_Pad1.33x1.80mm_HandSolder
- removed C2: 10uF, Capacitor_SMD:C_1206_3216Metric_Pad1.33x1.80mm_HandSolder
- added C10: 330uF, Capacitor_SMD:C_1206_3216Metric_Pad1.33x1.80mm_HandSolder, F.Cu at (190.6, 78.3)
- added C11: 100uF, Capacitor_SMD:C_1206_3216Metric_Pad1.33x1.80mm_HandSolder, F.Cu at (190.6, 81.7)
- added C12: 330uF, Capacitor_SMD:C_1206_3216Metric_Pad1.33x1.80mm_HandSolder, F.Cu at (210.0, 91.0)
- added C5: 100uF, Capacitor_SMD:C_1206_3216Metric_Pad1.33x1.80mm_HandSolder, F.Cu at (248.5, 66.8)
- added C6: 330uF, Capacitor_SMD:C_1206_3216Metric_Pad1.33x1.80mm_HandSolder, F.Cu at (190.6, 65.0)
- added C7: 100uF, Capacitor_SMD:C_1206_3216Metric_Pad1.33x1.80mm_HandSolder, F.Cu at (190.6, 68.3)
- added C8: 330uF, Capacitor_SMD:C_1206_3216Metric_Pad1.33x1.80mm_HandSolder, F.Cu at (190.6, 71.7)
- added C9: 100uF, Capacitor_SMD:C_1206_3216Metric_Pad1.33x1.80mm_HandSolder, F.Cu at (190.6, 75.0)
- added D2: 1N5822, 1N5822:DIOAD2120W130L950D530P, F.Cu at (235.1, 66.0)
- added D3: 1N5822, 1N5822:DIOAD2120W130L950D530P, F.Cu at (237.8, 81.2)
- added D4: 1N5822, 1N5822:DIOAD2120W130L950D530P, F.Cu at (181.3, 91.3)
- added D5: 1N5822, 1N5822:DIOAD2120W130L950D530P, F.Cu at (55.9, 86.6)
- added J2: USB_A, Connector_USB:USB_A_Molex_67643_Horizontal, F.Cu at (159.0, 68.4)
- added J3: USB_A, Connector_USB:USB_A_Molex_67643_Horizontal, F.Cu at (152.0, 119.2)
- added R1: 1K, Resistor_SMD:R_1206_3216Metric_Pad1.30x1.75mm_HandSolder, F.Cu at (215.3, 95.8)
- added R2: 3.09K, Resistor_SMD:R_1206_3216Metric_Pad1.30x1.75mm_HandSolder, F.Cu at (248.3, 72.1)
- added R3: 3.09K, Resistor_SMD:R_1206_3216Metric_Pad1.30x1.75mm_HandSolder, F.Cu at (215.3, 102.4)
- added R4: 1K, Resistor_SMD:R_1206_3216Metric_Pad1.30x1.75mm_HandSolder, F.Cu at (215.3, 105.7)
- added R5: 3.09K, Resistor_SMD:R_1206_3216Metric_Pad1.30x1.75mm_HandSolder, F.Cu at (215.3, 109.0)
- added R6: 1K, Resistor_SMD:R_1206_3216Metric_Pad1.30x1.75mm_HandSolder, F.Cu at (248.8, 84.9)
- added R7: 3.09K, Resistor_SMD:R_1206_3216Metric_Pad1.30x1.75mm_HandSolder, F.Cu at (215.3, 115.7)
- added R8: 1K, Resistor_SMD:R_1206_3216Metric_Pad1.30x1.75mm_HandSolder, F.Cu at (215.3, 119.0)
- added U2: LM2576-5.0WU, LM2576-5.0WU:MICROCHIP_TO-263, F.Cu at (266.2, 68.7)
- added U3: LM2576-5.0WU, LM2576-5.0WU:MICROCHIP_TO-263, F.Cu at (264.3, 115.4)
- added U4: LM2576-5.0WU, LM2576-5.0WU:MICROCHIP_TO-263, F.Cu at (268.9, 83.9)
- added U5: LM2576-5.0WU, LM2576-5.0WU:MICROCHIP_TO-263, F.Cu at (209.7, 108.5)
- D1: value D -> 1N5822; footprint Diode_SMD:D_1210_3225Metric_Pad1.42x2.65mm_HandSolder -> 1N5822:DIOAD2120W130L950D530P
- moved D1 197.5 mm to (237.5, 114.1)
- moved C3 42.4 mm to (122.8, 87.6)
- moved C4 42.4 mm to (126.5, 87.5)
- moved J1 42.4 mm to (68.1, 70.3)
- moved U1 42.4 mm to (73.0, 86.6)
Connections:
- net GND1 renamed -VDC
- U1 pad 1: Net-(D1-K) -> Net-(U1-+VIN(VCC))
Routing:
- net Net-(J2-D-): track 0.00 -> 59.3 mm
- net Net-(J2-VBUS): track 0.00 -> 53.7 mm
- net Net-(J2-D+): track 0.00 -> 51.6 mm
- net GND: track 0.00 -> 15.6 mm
- net Net-(D1-K): track 14.5 -> 0.00 mm
- net Net-(U2-OUTPUT): track 0.00 -> 8.57 mm
- net Net-(U1-+VIN(VCC)): track 0.00 -> 6.50 mm
- net +12V: track 11.5 -> 16.8 mm
- net Net-(U2-FEEDBACK): track 0.00 -> 4.49 mm
Other:
- board outline added: 241.6 x 69.3 mm
