File: ROCSAR_Hardware/Interface_PCB/Interface_PCB.kicad_pcb (KiCad board)
At the start: 2 copper layers, 175 x 100 mm, 86 parts, among them IC1 SN74LVC1G123DCTT, IC2 SN74LVC1G123DCTT, J1 1803277, J10 1803277, J11 1803277, J12 1803277, J13 Conn_01x02_Pin, J14 Conn_01x02_Pin, J2 1757242, J3 Conn_01x02_Pin, J4 RJE05188051C, J5 RJE05188051C, J6 USB1086-GF-B, J7 USB1086-GF-B, J8 Conn_01x02_Pin, J9 1803277, Q1 PBSS5250PAS-QX, Q2 PBSS5250PAS-QX, Q3 PBSS5250PAS-QX, Q4 SIHFR9024, Q5 SIHFR9024, U1 TEN 60-2422N, U2 LM2576-5.0WU, U3 LM2576-5.0WU, U6 SN74HC126PWR, U7 LM2576-5.0WU, U8 BNO055

Commit message: interface PCB
Parts:
- removed C1, C5: 100uF, Capacitor_SMD:C_1206_3216Metric_Pad1.33x1.80mm_HandSolder
- removed C15: 1uF, Capacitor_SMD:C_0603_1608Metric_Pad1.08x0.95mm_HandSolder
- removed C16: 100nF, Capacitor_SMD:C_0603_1608Metric_Pad1.08x0.95mm_HandSolder
- removed C17: 120nF, Capacitor_SMD:C_0603_1608Metric_Pad1.08x0.95mm_HandSolder
- removed C2, C6: 330uF, Capacitor_SMD:C_1206_3216Metric_Pad1.33x1.80mm_HandSolder
- removed D1, D2: 1N5822, 1N5822:DIOAD2120W130L950D530P
- removed J10, J11, J9: 1803277, 1803277:PHOENIX_1803277
- removed L1, L2, L5: 330uH, SRR1050HA-331Y:INDPM102100X510N
- removed R1, R23, R4: 1K, Resistor_SMD:R_1206_3216Metric_Pad1.30x1.75mm_HandSolder
- removed R2, R22, R3: 3.09K, Resistor_SMD:R_1206_3216Metric_Pad1.30x1.75mm_HandSolder
- removed R40, R41: 10K, Resistor_SMD:R_0603_1608Metric_Pad0.98x0.95mm_HandSolder
- removed U3, U7: LM2576-5.0WU, LM2576-5.0WU:MICROCHIP_TO-263
- removed U8: BNO055, BNO055:LGA28R50P4X10_380X520X100
- added D7: V10P6HM3_A_H, V10P6HM3_A_H:V10P6HM3_AH, F.Cu at (85.5, 108.5)
- added D8: V10P6HM3_A_H, V10P6HM3_A_H:V10P6HM3_AH, F.Cu at (94.7, 108.5)
- added J15: 1803277, 1803277:PHOENIX_1803277, F.Cu at (144.7, 36.0)
- added J16: 1803277, 1803277:PHOENIX_1803277, F.Cu at (134.5, 36.0)
- added PS1: TDN_3-1211WI, TDN_3-1211WI:TDN52412WI, F.Cu at (118.0, 107.5)
- added R42: 0, Resistor_SMD:R_0603_1608Metric_Pad0.98x0.95mm_HandSolder, F.Cu at (173.7, 90.0)
- C7: value 100uF -> 0.1uF
- C8: value 330uF -> 10uF
- D6: value 1N5822 -> V10P6HM3_A_H; footprint 1N5822:DIOAD2120W130L950D530P -> V10P6HM3_A_H:V10P6HM3_AH; moved to B.Cu
- U2: value LM2576-5.0WU -> ~; footprint LM2576-5.0WU:MICROCHIP_TO-263 -> AdafruitBNO055:Adafruit BNO055
- moved U2 91.5 mm to (162.1, 120.6)
- moved C7 59.1 mm to (128.5, 106.7)
- moved C8 54.0 mm to (128.5, 110.5), turned to 0 degrees
- moved D6 52.6 mm to (115.7, 118.5), turned to 180 degrees
Connections:
- A1 pad 11: unconnected-(A1-GPIO8-Pad11) -> BNO_PS1
- A1 pad 12: unconnected-(A1-GPIO9-Pad12) -> BNO_PS0
- A1 pad 16: SDA / UART TX -> BNO_SDA
- A1 pad 17: SCL / UART RX -> BNO_SCL
- A1 pad 24: N_RESET -> BNO_RST
- A1 pad 25: INT -> BNO_INT
- A1 pad 29: I2C_ADDR_SEL -> BNO_ADDR
- A1 pad 31: ON/OFF 0 -> unconnected-(A1-GPIO26_ADC0-Pad31)
- A1 pad 32: ON/OFF 1 -> unconnected-(A1-GPIO27_ADC1-Pad32)
- A1 pad 39: +5V Main -> +5V
- C7 pad 1: +12V -> +5V
- C8 pad 1: GND -> +5V
- C8 pad 2: +5V Servo -> GND
- IC1 pad 2: +5V Main -> +5V
- IC1 pad 3: +5V Main -> +5V
- IC1 pad 8: +5V Main -> +5V
- IC2 pad 2: +5V Servo -> +5V
- IC2 pad 3: +5V Servo -> +5V
- IC2 pad 8: +5V Servo -> +5V
- J1 pad 01: Net-(U1-REMOTE_ON/OFF) -> -VDC
- J1 pad 02: -VDC -> Net-(D7-A_1)
- J12 pad 01: +VDC -> +12V
- J12 pad 02: -VDC -> GND
- R14 pad 1: +5V Main -> +5V
- R19 pad 2: +5V Main -> +5V
- R24 pad 1: +5V Main -> +5V
- R30 pad 1: +5V Main -> +5V
- R33 pad 1: +5V Servo -> +5V
- R36 pad 1: +5V Servo -> +5V
- R9 pad 1: +5V Main -> +5V
- U1 pad 3: Net-(U1-REMOTE_ON/OFF) -> ON/OFF
- U2 pad 1: +12V -> +3.3V
- U2 pad 2: Net-(U2-OUTPUT) -> unconnected-(U2-3vo-Pad2)
- U2 pad 4: Net-(U2-FEEDBACK) -> BNO_SDA
- U2 pad 5: GND -> BNO_SCL
- U2 pad 6: GND -> BNO_RST
- U6 pad 14: +5V Main -> +5V
Routing:
- net +5V: track 0.00 -> 281.6 mm, vias 0 -> 5
- net +5V Main: track 189.9 -> 0.00 mm, vias 4 -> 0
- net +5V Servo: track 140.8 -> 0.00 mm, vias 4 -> 0
- net GND: track 169.7 -> 57.5 mm, vias 58 -> 22
- net +12V: track 249.9 -> 159.0 mm, vias 7 -> 4
- net +VDC: track 104.6 -> 28.5 mm
- net BNO_SCL: track 0.00 -> 65.5 mm
- net SCL / UART RX: track 57.3 -> 0.00 mm, vias 2 -> 0
- net BNO_SDA: track 0.00 -> 54.4 mm, vias 0 -> 1
- net BNO_RST: track 0.00 -> 50.9 mm, vias 0 -> 1
- net +5V GNSS: track 50.0 -> 0.00 mm
- net BNO_PS0: track 0.00 -> 49.8 mm, vias 0 -> 1
- net SDA / UART TX: track 46.3 -> 0.00 mm, vias 4 -> 0
- net BNO_PS1: track 0.00 -> 42.5 mm
- net ON/OFF: track 0.00 -> 41.6 mm
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
Commit message: interface changes
Parts:
- added J10: 1723103103, 1723103103:MOLEX_1723103103, F.Cu at (137.5, 122.3)
- added J9: 1723103103, 1723103103:MOLEX_1723103103, F.Cu at (120.8, 122.3)
Routing:
- net +12V: track 159.0 -> 254.4 mm
- net SERVO_OUT: track 0.00 -> 79.8 mm, vias 0 -> 1
- net -VDC: track 120.6 -> 114.4 mm
