File: ROCSAR_Hardware/Interface_PCB/Interface_PCB.kicad_pcb (KiCad board)
At the start: 2 copper layers, 175 x 100 mm, 68 parts, among them IC1 SN74LVC1G123DCTT, IC2 SN74LVC1G123DCTT, J1 1803277, J10 1723103103, J12 1803277, J13 Conn_01x02_Pin, J14 Conn_01x02_Pin, J15 1803277, J16 1803277, J2 1757242, J3 Conn_01x02_Pin, J4 RJE05188051C, J5 RJE05188051C, J6 USB1086-GF-B, J7 USB1086-GF-B, J8 Conn_01x02_Pin, J9 1723103103, Q1 PBSS5250PAS-QX, Q2 PBSS5250PAS-QX, Q3 PBSS5250PAS-QX, Q4 SIHFR9024, Q5 SIHFR9024, U1 TEN 60-2422N, U6 SN74HC126PWR

Commit message: interface
Parts:
- J12, J15, J16: moved to B.Cu
- moved J12 7.74 mm to (89.8, 35.9), turned to 0 degrees
- turned J15 to 0 degrees
- turned J16 to 0 degrees
Routing:
- net +12V: track 254.4 -> 258.2 mm
- net +5V: track 281.6 -> 278.9 mm

Commit message: pcb
Parts:
- removed C14: C_Small, Capacitor_SMD:C_0603_1608Metric_Pad1.08x0.95mm_HandSolder
- added C15: C_Small, Capacitor_THT:C_Radial_D10.0mm_H16.0mm_P5.00mm, F.Cu at (180.5, 64.5)
- C13: footprint Capacitor_SMD:C_0603_1608Metric_Pad1.08x0.95mm_HandSolder -> Capacitor_THT:C_Radial_D10.0mm_H16.0mm_P5.00mm
- moved C13 15.3 mm to (205.5, 62.5), turned to 90 degrees
- moved G*** 5.14 mm to (176.4, 78.7)
Routing:
- net Net-(IC1-REXT/CEXT): track 13.2 -> 22.2 mm
- net Net-(IC2-REXT/CEXT): track 11.8 -> 15.6 mm
- net GND: track 57.5 -> 56.0 mm, vias 22 -> 21
Other:
- board text added: "-Simular SN74LVC1G123DCTT em spice -Mudar condensador do SN74LVC1G123DCTT para DIP"
