File: ROCSAR_Hardware/Interface_PCB/Interface_PCB.kicad_sch (KiCad schematic)
At the start: 7 parts, among them J1 Remove Before Flight, U1 TEN 60-2422N

Commit message: PCB Update
Parts:
- removed C1: 0.1uF, Capacitor_SMD:C_1206_3216Metric_Pad1.33x1.80mm_HandSolder, symbol Device:C
- removed C2: 10uF, Capacitor_SMD:C_1206_3216Metric_Pad1.33x1.80mm_HandSolder, symbol Device:C
- removed D1: D, Diode_SMD:D_1210_3225Metric_Pad1.42x2.65mm_HandSolder, symbol Device:D
- added C10, C12, C6, C8: 330uF, Capacitor_SMD:C_1206_3216Metric_Pad1.33x1.80mm_HandSolder, symbol Device:C
- added C11, C5, C7, C9: 100uF, Capacitor_SMD:C_1206_3216Metric_Pad1.33x1.80mm_HandSolder, symbol Device:C
- added D1, D2, D3, D4, D5: 1N5822, 1N5822:DIOAD2120W130L950D530P, symbol 1N5822:1N5822
- added J2, J3: USB_A, Connector_USB:USB_A_Molex_67643_Horizontal, symbol Connector:USB_A
- added L1, L2, L3, L4: 100uH, symbol Device:L
- added R1, R4, R6, R8: 1K, Resistor_SMD:R_1206_3216Metric_Pad1.30x1.75mm_HandSolder, symbol Device:R
- added R2, R3, R5, R7: 3.09K, Resistor_SMD:R_1206_3216Metric_Pad1.30x1.75mm_HandSolder, symbol Device:R
- added U2, U3, U4, U5: LM2576-5.0WU, LM2576-5.0WU:MICROCHIP_TO-263, symbol LM2576-5_0WU:LM2576-5.0WU
- J1: footprint (none) -> Connector_PinHeader_2.54mm:PinHeader_1x02_P2.54mm_Vertical
Connections:
- net +12V: now also C11.1, C5.1, C7.1, C9.1, U2.1 (VIN), U3.1 (VIN), U4.1 (VIN), U5.1 (VIN)
- net GND: now also C10.1, C11.2, C12.1, C5.2, C6.1, C7.2, C8.1, C9.2, D1.A, D2.A, D3.A, D4.A, J2.4 (GND), J3.4 (GND), R1.2, R4.2, R6.2, R8.2, U2.3 (GROUND), U2.5 (~{ON}/OFF), U2.6 (GND), U3.3 (GROUND), U3.5 (~{ON}/OFF), U3.6 (GND), U4.3 (GROUND), U4.5 (~{ON}/OFF), U4.6 (GND), U5.3 (GROUND), U5.5 (~{ON}/OFF), U5.6 (GND)
- net at U1.1 (+VIN(VCC)): now also D5.C
- net GND1 renamed -VDC
- new net: D4.C, L4.2, U5.2 (OUTPUT)
- new net: R7.2, R8.1, U5.4 (FEEDBACK)
- new net: R3.2, R4.1, U3.4 (FEEDBACK)
- new net: D1.C, L2.2, U3.2 (OUTPUT)
- new net: R1.1, R2.2, U2.4 (FEEDBACK)
- new net: D3.C, L3.2, U4.2 (OUTPUT)
- new net: R5.2, R6.1, U4.4 (FEEDBACK)
- new net: J2.1 (VBUS), J3.1 (VBUS)
- new net: J2.2 (D-), J3.2 (D-)
- new net: J2.3 (D+), J3.3 (D+)
- new net: D2.C, L1.2, U2.2 (OUTPUT)
- new net +5V: C10.2, C12.2, C6.2, C8.2, L1.1, L2.1, L3.1, L4.1, R2.1, R3.1, R5.1, R7.1
- new net +VDC: D5.A
Other:
- note added: "Power Regulation System - VDC-12V (12V-5V * 4)"
- note added: "Vout = 1.23*(1+(R2/R1))"
- note added: "X"
- note removed: "Traco Power"
- moved on the sheet: C3, C4, J1, U1
