File: ROCSAR_Hardware/Interface_PCB/Interface_PCB.kicad_sch (KiCad schematic)
At the start: 35 parts, among them J1 Remove Before Flight, J2 USB_A, J3 USB_A, U1 TEN 60-2422N, U2 LM2576-5.0WU, U3 LM2576-5.0WU, U4 LM2576-5.0WU, U5 LM2576-5.0WU

Commit message: Continuation of the development of the interface pcb
Parts:
- L1, L2, L3, L4: value 100uH -> 330uH; footprint (none) -> SRR1050HA-331Y:INDPM102100X510N
Connections:
- removed net +5V: C10.2, C12.2, C6.2, C8.2, L1.1, L2.1, L3.1, L4.1, R2.1, R3.1, R5.1, R7.1
- new net: C8.2, L2.1, R3.1
- new net: C6.2, L1.1, R2.1
- new net: C10.2, L3.1, R5.1
- new net: C12.2, L4.1, R7.1
- no-connect marks 0 -> 2
Other:
- note added: "USB Connection"
- moved on the sheet: J2, J3

Commit message: Interface PCB mostly done
Parts:
- removed D5: 1N5822, 1N5822:DIOAD2120W130L950D530P, symbol 1N5822:1N5822
- removed J1: Remove Before Flight, Connector_PinHeader_2.54mm:PinHeader_1x02_P2.54mm_Vertical, symbol Connector:Conn_01x02_Pin
- removed J2, J3: USB_A, Connector_USB:USB_A_Molex_67643_Horizontal, symbol Connector:USB_A
- added A1: RaspberryPi_Pico, Module:RaspberryPi_Pico_Common_Unspecified, symbol MCU_Module:RaspberryPi_Pico
- added C1: 100uF, Capacitor_SMD:C_1206_3216Metric_Pad1.33x1.80mm_HandSolder, symbol Device:C
- added C13, C14: C_Small, Capacitor_SMD:C_0603_1608Metric_Pad1.08x0.95mm_HandSolder, symbol Device:C_Small
- added C15: 1uF, Capacitor_SMD:C_0603_1608Metric_Pad1.08x0.95mm_HandSolder, symbol Device:C_Small
- added C16: 100nF, Capacitor_SMD:C_0603_1608Metric_Pad1.08x0.95mm_HandSolder, symbol Device:C_Small
- added C17: 120nF, Capacitor_SMD:C_0603_1608Metric_Pad1.08x0.95mm_HandSolder, symbol Device:C_Small
- added C2: 330uF, Capacitor_SMD:C_1206_3216Metric_Pad1.33x1.80mm_HandSolder, symbol Device:C
- added D5: V10P6HM3_A_H, V10P6HM3_AH, symbol V10P6HM3_A_H:V10P6HM3_A_H
- added D6: 1N5822, 1N5822:DIOAD2120W130L950D530P, symbol 1N5822:1N5822
- added IC1, IC2: SN74LVC1G123DCTT, SOP65P400X130-8N, symbol SN74LVC1G123DCTT:SN74LVC1G123DCTT
- added J1: 1803277, PHOENIX_1803277, symbol 1803277:1803277
- added J2: 1757242, PHOENIX_1757242, symbol 1757242:1757242
- added J4, J5: RJE05188051C, RJE05188051C, symbol RJE05188051C:RJE05188051C
- added J6, J7: USB1086-GF-B, USB1086GFB, symbol USB1086-GF-B:USB1086-GF-B
- added JP1: Jumper_2_Open, Jumper:SolderJumper-2_P1.3mm_Open_RoundedPad1.0x1.5mm, symbol Jumper:Jumper_2_Open
- added L5: 330uH, SRR1050HA-331Y:INDPM102100X510N, symbol Device:L
- added Q1, Q2, Q3: PBSS5250PAS-QX, PMEG2020EPASX, symbol PBSS5250PAS-QX:PBSS5250PAS-QX
- added R10, R25, R35: 100K, Resistor_SMD:R_0603_1608Metric_Pad0.98x0.95mm_HandSolder, symbol Device:R_Small
- added R11, R18, R26, R37, R40, R41, R9: 10K, Resistor_SMD:R_0603_1608Metric_Pad0.98x0.95mm_HandSolder, symbol Device:R_Small
- added R12: 22K, Resistor_SMD:R_0603_1608Metric_Pad0.98x0.95mm_HandSolder, symbol Device:R_Small
- added R13, R15, R16, R21: 2K2, Resistor_SMD:R_0603_1608Metric_Pad0.98x0.95mm_HandSolder, symbol Device:R_Small
- added R14, R17: 5K6, Resistor_SMD:R_0603_1608Metric_Pad0.98x0.95mm_HandSolder, symbol Device:R_Small
- added R19, R20: NI, Resistor_SMD:R_0603_1608Metric_Pad0.98x0.95mm_HandSolder, symbol Device:R_Small
- added R22: 3.09K, Resistor_SMD:R_1206_3216Metric_Pad1.30x1.75mm_HandSolder, symbol Device:R
- added R23: 1K, Resistor_SMD:R_1206_3216Metric_Pad1.30x1.75mm_HandSolder, symbol Device:R
- added R24, R30, R31, R32, R33, R36: R_Small, Resistor_SMD:R_0603_1608Metric_Pad0.98x0.95mm_HandSolder, symbol Device:R_Small
- added R27, R39: 4K7, Resistor_SMD:R_0603_1608Metric_Pad0.98x0.95mm_HandSolder, symbol Device:R_Small
- added R28, R38: 3K3, Resistor_SMD:R_0603_1608Metric_Pad0.98x0.95mm_HandSolder, symbol Device:R_Small
- added R29, R34: ~, Resistor_SMD:R_0603_1608Metric_Pad0.98x0.95mm_HandSolder, symbol Device:R_Small
- added R42, R43: TBD, Resistor_SMD:R_0603_1608Metric_Pad0.98x0.95mm_HandSolder, symbol Device:R_Small
- added U6: SN74HC126PWR, PW14, symbol PW14:SN74HC126PWR
- added U7: LM2576-5.0WU, LM2576-5.0WU:MICROCHIP_TO-263, symbol LM2576-5_0WU:LM2576-5.0WU
- added U8: BNO055, BNO055:LGA28R50P4X10_380X520X100, symbol BNO055:BNO055
Connections:
- net +12V: now also C1.1, R28.2, R38.2, U7.1 (VIN)
- net +VDC: now also D5.1 (A_1), D5.2 (A_2), J2.02
- net -VDC: now also J1.02, J2.01
- net GND: now also A1.13 (GND), A1.18 (GND), A1.23 (GND), A1.28 (GND), A1.3 (GND), A1.38 (GND), A1.8 (GND), C1.2, C13.2, C14.2, C15.2, C16.2, C17.2, C2.1, D6.A, IC1.4 (GND), IC1.6 (CEXT), IC2.4 (GND), IC2.6 (CEXT), JP1.1 (A), Q1.2 (E), Q2.2 (E), Q3.2 (E), R10.2, R18.2, R20.1, R23.2, R25.2, R29.2, R34.2, R35.2, U6.7 (GND), U7.3 (GROUND), U7.5 (~{ON}/OFF), U7.6 (GND), U8.18 (COM2), U8.2 (GND), U8.25 (GNDIO), U8.5 (PS1), U8.6 (PS0)
- net +5V Servo: now reaches C8.2, L2.1, R3.1
- net +5V Servo: now also IC1.2 (B), IC1.3 (~{CLR}), IC1.8 (VCC), IC2.2 (B), IC2.3 (~{CLR}), IC2.8 (VCC), R24.1, R30.1, R33.1, R36.1
- net +5V GNSS: now reaches C6.2, L1.1, R2.1
- net at U1.1 (+VIN(VCC)): now also D5.3 (K)
- net at U1.3 (REMOTE_ON/OFF): now also J1.01
- net +5V RX: now reaches C10.2, L3.1, R5.1
- net +5V TX: now reaches C12.2, L4.1, R7.1
- new net: IC2.1 (~{A}), R32.2, R33.2, R34.1
- new net: Q2.1 (B), R11.2
- new net: Q2.3 (C_1), Q2.4 (C_2), R14.2, R15.2
- new net: J6.1 (VBUS), J7.1 (VBUS)
- new net: J6.10 (MH1), J7.10 (MH1)
- new net: J6.11 (MH2), J7.11 (MH2)
- new net: J6.2 (D-), J7.2 (D-)
- new net: J6.3 (D+), J7.3 (D+)
- new net: J6.4 (GND), J7.4 (GND)
- new net: J6.5 (STDA_SSRX-), J7.5 (STDA_SSRX-)
- new net: J6.6 (STDA_SSRX+), J7.6 (STDA_SSRX+)
- new net: J6.7 (GND_DRAIN), J7.7 (GND_DRAIN)
- new net: J6.8 (STDA_SSTX-), J7.8 (STDA_SSTX-)
- new net: J6.9 (STDA_SSTX+), J7.9 (STDA_SSTX+)
- new net: R15.1, R16.1, U6.4 (2OE)
- new net: J4.1, J5.1
- new net: J4.2, J5.2
- new net: J4.3, J5.3
- new net: J4.4, J5.4
- new net: J4.5, J5.5
- new net: J4.6, J5.6
- new net: J4.7, J5.7
- new net: J4.8, J5.8
- new net: R21.1, U6.3 (1Y)
- new net: IC1.1 (~{A}), R29.1, R30.2, R31.2
- new net: R22.2, R23.1, U7.4 (FEEDBACK)
- new net: R10.1, R11.1, R12.2
- new net: JP1.2 (B), R40.1, U8.4 (NBOOT_LOAD_PIN)
- new net: C15.1, U8.9 (CAP)
- new net: IC1.5 (Q), R25.1, R26.1
- new net: Q1.1 (B), R26.2
- new net: Q1.3 (C_1), Q1.4 (C_2), R27.1
- new net: C14.1, IC2.7 (REXT/CEXT), R36.2
- new net: R27.2, R28.1
- new net: C13.1, IC1.7 (REXT/CEXT), R24.2
- new net: IC2.5 (Q), R35.1, R37.1
- new net: Q3.1 (B), R37.2
- new net: R38.1, R39.2
- new net: D6.C, L5.2, U7.2 (OUTPUT)
- new net: R17.1, U6.6 (2Y)
- new net: Q3.3 (C_1), Q3.4 (C_2), R39.1
- new net: R13.2, R19.1, R20.2, U6.2 (1A)
- new net +3.3V: A1.36 (3V3), C16.1, C17.1, R40.2, R41.2, R42.1, R43.1, U8.28 (VDDIO), U8.3 (VDD)
- new net +5V Main: A1.39 (VSYS), C2.2, L5.1, R14.1, R19.2, R22.1, R9.1, U6.14 (VCC)
- new net BL_IND: U8.10 (PIN10)
- new net I2C_ADDR_SEL: U8.17 (COM3)
- new net INT: U8.14 (INT)
- new net MCU_HEAT_1: R31.1
- new net MCU_HEAT_2: R32.1
- new net N_RESET: R41.1, U8.11 (NRESET)
- new net RX_EN: R16.2
- new net SCL: R42.2, U8.20 (COM0)
- new net SDA: R43.2, U8.19 (COM1)
- new net SERVO_OUT: R21.2, R9.2, U6.5 (2A)
- new net TX_EN: R12.1, U6.1 (1OE)
- new net UART RX: R17.2, R18.1
- new net UART TX: R13.1
- no-connect marks 2 -> 10
Other:
- note added: "3 pins"
- note added: "4 pins"
- note added: "BNO055 IMU"
- note added: "Ethernet Connection"
- note added: "GNSS Buck"
- note added: "Main Buck"
- note added: "Power Regulation System - VDC-12V (12V-5V * 5)"
- note added: "RF RX Buck"
- note added: "RF TX Buck"
- note added: "Raspberry Pi PICO"
- note added: "Servo Buck"
- note added: "Servo Heaters"
- note added: "UART Buffer"
- note removed: "Power Regulation System - VDC-12V (12V-5V * 4)"
- moved on the sheet: C10, C11, C12, C5, C6, C7, C8, C9, D1, D2, D3, D4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

Commit message: atualizacoes interface
Parts:
- added J10, J3, J8, J9: 1803277, PHOENIX_1803277, symbol 1803277:1803277
- added Q4, Q5: SIHFR9024, SIHFR9024:SIHFR9024, symbol Transistor_FET:BS108
Connections:
- net +12V: now also Q4.1 (D), Q5.1 (D)
- net +5V Main: now also J10.01
- net +5V RX: now also J3.01
- net +5V Servo: now also J9.01
- net +5V TX: now also J8.01
- net GND: now also J10.02, J3.02, J8.02, J9.02
- net I2C_ADDR_SEL: now also A1.29 (GPIO22)
- net INT: now also A1.25 (GPIO19)
- net MCU_HEAT_1: now also A1.22 (GPIO17)
- net MCU_HEAT_2: now also A1.21 (GPIO16)
- net N_RESET: now also A1.24 (GPIO18)
- net RX_EN: now also A1.14 (GPIO10)
- net SCL: now also A1.32 (GPIO27_ADC1)
- net SDA: now also A1.31 (GPIO26_ADC0)
- net TX_EN: now also A1.15 (GPIO11)
- net UART RX: now also A1.27 (GPIO21)
- net UART TX: now also A1.26 (GPIO20)
- net at R27.2, R28.1: now also Q4.2 (G)
- net at R38.1, R39.2: now also Q5.2 (G)
- new net Heating 1: Q4.3 (S)
- new net Heating 2: Q5.3 (S)
Other:
- note added: "Nao sei como conectar a inteface --->"
- moved on the sheet: C10, C11, C12, C2, C8, C9, D3, D4, L3, L4, R28, R5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

Commit message: Interface
Parts:
- removed JP1: Jumper_2_Open, Jumper:SolderJumper-2_P1.3mm_Open_RoundedPad1.0x1.5mm, symbol Jumper:Jumper_2_Open
- removed R42, R43: TBD, Resistor_SMD:R_0603_1608Metric_Pad0.98x0.95mm_HandSolder, symbol Device:R_Small
- added J11: 1803277, PHOENIX_1803277, symbol 1803277:1803277
Connections:
- net +5V GNSS: now also J11.01
- net GND: now also J11.02; no longer U8.5 (PS1), U8.6 (PS0)
- net SDA / UART TX: now reaches A1.16 (GPIO12)
- net SDA / UART TX: now also U8.19 (COM1)
- net SCL / UART RX: now reaches A1.17 (GPIO13)
- net SCL / UART RX: now also U8.20 (COM0)
- net SCL renamed ON/OFF 1
- net ON/OFF 1: now also U8.5 (PS1); no longer U8.20 (COM0)
- net SDA renamed ON/OFF 0
- net ON/OFF 0: now also U8.6 (PS0); no longer U8.19 (COM1)
Other:
- note added: "Interface PCB"
- note removed: "Nao sei como conectar a inteface --->"
- moved on the sheet: C6, R40, R41

Commit message: Interface Updates
Parts:
- removed C10, C12: 330uF, Capacitor_SMD:C_1206_3216Metric_Pad1.33x1.80mm_HandSolder, symbol Device:C
- removed C11, C9: 100uF, Capacitor_SMD:C_1206_3216Metric_Pad1.33x1.80mm_HandSolder, symbol Device:C
- removed D3, D4: 1N5822, 1N5822:DIOAD2120W130L950D530P, symbol 1N5822:1N5822
- removed J3, J8: 1803277, PHOENIX_1803277, symbol 1803277:1803277
- removed L3, L4: 330uH, SRR1050HA-331Y:INDPM102100X510N, symbol Device:L
- removed R5, R7: 3.09K, Resistor_SMD:R_1206_3216Metric_Pad1.30x1.75mm_HandSolder, symbol Device:R
- removed R6, R8: 1K, Resistor_SMD:R_1206_3216Metric_Pad1.30x1.75mm_HandSolder, symbol Device:R
- removed U4, U5: LM2576-5.0WU, LM2576-5.0WU:MICROCHIP_TO-263, symbol LM2576-5_0WU:LM2576-5.0WU
- added J12: 1803277, PHOENIX_1803277, symbol 1803277:1803277
- added J13, J14, J3, J8: Conn_01x02_Pin, Connector_PinHeader_2.54mm:PinHeader_1x02_P2.54mm_Vertical, symbol Connector:Conn_01x02_Pin
- added R42: 0, symbol Device:R
- R9: value 10K -> 1M
Connections:
- net +5V Main: now also IC1.2 (B), IC1.3 (~{CLR}), IC1.8 (VCC), R24.1, R30.1
- net +5V Servo: no longer IC1.2 (B), IC1.3 (~{CLR}), IC1.8 (VCC), R24.1, R30.1
- net +VDC: now also J12.01
- net -VDC: now also J12.02
- net SERVO_OUT: now also R42.1; no longer R21.2, R9.2, U6.5 (2A)
- new net: R21.2, R42.2, R9.2, U6.5 (2A)
- new net: J13.2 (Pin_2), J14.1 (Pin_1)
- new net: J13.1 (Pin_1), J14.2 (Pin_2)
- new net: J3.2 (Pin_2), J8.1 (Pin_1)
- new net: J3.1 (Pin_1), J8.2 (Pin_2)
Other:
- note added: "-12v -gnd -toggle"
- note added: "Fan Power 1"
- note added: "Fan Power 2"
- note removed: "RF RX Buck"
- note removed: "RF TX Buck"
- moved on the sheet: C5, C6, D2, J11, L1, R1, R2, U2
