File: ROCSAR_Hardware/Interface_PCB/Interface_PCB.kicad_sch (KiCad schematic)
At the start: 86 parts, among them IC1 SN74LVC1G123DCTT, IC2 SN74LVC1G123DCTT, J1 1803277, J10 1803277, J11 1803277, J12 1803277, J13 Conn_01x02_Pin, J14 Conn_01x02_Pin, J2 1757242, J3 Conn_01x02_Pin, J4 RJE05188051C, J5 RJE05188051C, J6 USB1086-GF-B, J7 USB1086-GF-B, J8 Conn_01x02_Pin, J9 1803277, Q1 PBSS5250PAS-QX, Q2 PBSS5250PAS-QX, Q3 PBSS5250PAS-QX, Q4 SIHFR9024, Q5 SIHFR9024, U1 TEN 60-2422N, U2 LM2576-5.0WU, U3 LM2576-5.0WU, U6 SN74HC126PWR, U7 LM2576-5.0WU, U8 BNO055

Commit message: interface PCB
Parts:
- removed C1, C5, C7: 100uF, Capacitor_SMD:C_1206_3216Metric_Pad1.33x1.80mm_HandSolder, symbol Device:C
- removed C15: 1uF, Capacitor_SMD:C_0603_1608Metric_Pad1.08x0.95mm_HandSolder, symbol Device:C_Small
- removed C16: 100nF, Capacitor_SMD:C_0603_1608Metric_Pad1.08x0.95mm_HandSolder, symbol Device:C_Small
- removed C17: 120nF, Capacitor_SMD:C_0603_1608Metric_Pad1.08x0.95mm_HandSolder, symbol Device:C_Small
- removed C2, C6, C8: 330uF, Capacitor_SMD:C_1206_3216Metric_Pad1.33x1.80mm_HandSolder, symbol Device:C
- removed D1, D2, D6: 1N5822, 1N5822:DIOAD2120W130L950D530P, symbol 1N5822:1N5822
- removed J10, J11, J9: 1803277, PHOENIX_1803277, symbol 1803277:1803277
- removed L1, L2, L5: 330uH, SRR1050HA-331Y:INDPM102100X510N, symbol Device:L
- removed R1, R23, R4: 1K, Resistor_SMD:R_1206_3216Metric_Pad1.30x1.75mm_HandSolder, symbol Device:R
- removed R2, R22, R3: 3.09K, Resistor_SMD:R_1206_3216Metric_Pad1.30x1.75mm_HandSolder, symbol Device:R
- removed R40, R41: 10K, Resistor_SMD:R_0603_1608Metric_Pad0.98x0.95mm_HandSolder, symbol Device:R_Small
- removed U2, U3, U7: LM2576-5.0WU, LM2576-5.0WU:MICROCHIP_TO-263, symbol LM2576-5_0WU:LM2576-5.0WU
- removed U8: BNO055, BNO055:LGA28R50P4X10_380X520X100, symbol BNO055:BNO055
- added C7: 0.1uF, Capacitor_SMD:C_1206_3216Metric_Pad1.33x1.80mm_HandSolder, symbol Device:C_Small
- added C8: 10uF, Capacitor_SMD:C_1206_3216Metric_Pad1.33x1.80mm_HandSolder, symbol Device:C_Small
- added D6, D7, D8: V10P6HM3_A_H, V10P6HM3_AH, symbol V10P6HM3_A_H:V10P6HM3_A_H
- added PS1: TDN_3-1211WI, TDN52412WI, symbol TDN_3-1211WI:TDN_3-1211WI
- added U2: (no value), AdafruitBNO055:Adafruit BNO055, symbol AdafruitBNO055:AdafruitBNO055
- R29, R34: value ~ -> (none)
- R42: footprint (none) -> Resistor_SMD:R_0603_1608Metric_Pad0.98x0.95mm_HandSolder
Connections:
- net +5V Servo is gone; now on net +5V: IC2.2 (B), IC2.3 (~{CLR}), IC2.8 (VCC), R33.1, R36.1
- net +12V: now also J12.01
- net +3.3V: now also U2.1 (Vin)
- net +VDC: now also D6.1 (A_1), D6.2 (A_2); no longer J12.01
- net -VDC: now also J1.01, D8.1 (A_1), D8.2 (A_2), PS1.2 (-VIN_(GND)); no longer J1.02, J12.02
- net GND: now also J12.02, C7.2, C8.2, PS1.5 (-VOUT), U2.3 (GND)
- net ON/OFF: now reaches U1.3 (REMOTE_ON/OFF)
- net ON/OFF: now also D7.3 (K), D8.3 (K), PS1.4 (ON/OFF); no longer J1.01
- net BNO_PS1: now reaches A1.11 (GPIO8)
- net BNO_PS1: now also U2.8 (PS1)
- net BNO_PS0: now reaches A1.12 (GPIO9)
- net BNO_PS0: now also U2.7 (PS0)
- net +5V Main renamed +5V
- net +5V: now also C7.1, C8.1, PS1.7 (+VOUT)
- net I2C_ADDR_SEL renamed BNO_ADDR
- net BNO_ADDR: now also U2.10 (ADDR)
- net INT renamed BNO_INT
- net BNO_INT: now also U2.9 (INT)
- net N_RESET renamed BNO_RST
- net BNO_RST: now also U2.6 (RST)
- net ON/OFF 0: no longer names the net of A1.31 (GPIO26_ADC0)
- net ON/OFF 1: no longer names the net of A1.32 (GPIO27_ADC1)
- net SCL / UART RX renamed BNO_SCL
- net BNO_SCL: now also U2.5 (SCL)
- net SDA / UART TX renamed BNO_SDA
- net BNO_SDA: now also U2.4 (SDA)
- new net: D6.3 (K), PS1.1 (+VIN_(VCC))
- new net: D7.1 (A_1), D7.2 (A_2), J1.02
- no-connect marks 10 -> 7
Other:
- note added: "Power Regulation System - VDC-12V VDC-5V"
- note added: "Remove Before Flight"
- note removed: "GNSS Buck"
- note removed: "Main Buck"
- note removed: "Power Regulation System - VDC-12V (12V-5V * 5)"
- note removed: "Servo Buck"
- note removed: "Vout = 1.23*(1+(R2/R1))"
- moved on the sheet: J1, J12

Commit message: interface pcb
Parts:
- added J15, J16: 1803277, PHOENIX_1803277, symbol 1803277:1803277
Connections:
- net +5V: now also J15.01, J16.01
- net GND: now also J15.02, J16.02

Commit message: interface changes
Parts:
- added J10, J9: 1723103103, 1723103103:MOLEX_1723103103, symbol 1723103103:1723103103
Connections:
- net +12V: now also J10.1, J9.1
- net GND: now also J10.3, J10.S1 (SHIELD1), J10.S2 (SHIELD2), J9.3, J9.S1 (SHIELD1), J9.S2 (SHIELD2)
- net SERVO_OUT: now also J10.2, J9.2
Other:
- note added: "Servo Connectors"
- moved on the sheet: D7, D8, J1
