File: ROCSAR_Hardware/Interface_PCB/Interface_PCB.kicad_sch (KiCad schematic)
At the start: 67 parts, among them IC1 SN74LVC1G123DCTT, IC2 SN74LVC1G123DCTT, J1 1803277, J10 1723103103, J12 1803277, J13 Conn_01x02_Pin, J14 Conn_01x02_Pin, J15 1803277, J16 1803277, J2 1757242, J3 Conn_01x02_Pin, J4 RJE05188051C, J5 RJE05188051C, J6 USB1086-GF-B, J7 USB1086-GF-B, J8 Conn_01x02_Pin, J9 1723103103, Q1 PBSS5250PAS-QX, Q2 PBSS5250PAS-QX, Q3 PBSS5250PAS-QX, Q4 SIHFR9024, Q5 SIHFR9024, U1 TEN 60-2422N, U6 SN74HC126PWR

Commit message: pcb
Parts:
- removed C14: C_Small, Capacitor_SMD:C_0603_1608Metric_Pad1.08x0.95mm_HandSolder, symbol Device:C_Small
- added C15: C_Small, Capacitor_THT:C_Radial_D10.0mm_H16.0mm_P5.00mm, symbol Device:C_Small
- C13: footprint Capacitor_SMD:C_0603_1608Metric_Pad1.08x0.95mm_HandSolder -> Capacitor_THT:C_Radial_D10.0mm_H16.0mm_P5.00mm
Connections:
- net GND: now also C15.2
- net at IC2.7 (REXT/CEXT), R36.2: now also C15.1
Changed lines of the file:
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@@
 	)
 	(junction
+		(at 262.89 251.46)
+		(diameter 0)
+		(color 0 0 0 0)
+	)
+	(junction
 		(at 184.15 180.4664)
 		(diameter 0)
@@
 	)
 	(junction
+		(at 262.89 246.38)
+		(diameter 0)
+		(color 0 0 0 0)
+	)
+	(junction
 		(at 261.62 261.62)
 		(diameter 0)
@@
 	)
 	(junction
-		(at 262.89 251.46)
-		(diameter 0)
-		(color 0 0 0 0)
-	)
-	(junction
-		(at 262.89 246.38)
-		(diameter 0)
-		(color 0 0 0 0)
-	)
-	(junction
 		(at 207.01 236.22)
 		(diameter 0)
@@
 	)
 	(junction
+		(at 251.46 123.19)
+		(diameter 0)
+		(color 0 0 0 0)
+	)
+	(junction
 		(at 74.93 152.4)
 		(diameter 0)
@@
 		)
 	)
+	(wire
+		(pts
+			(xy 251.46 123.19) (xy 254 123.19)
+		)
+		(stroke
+			(width 0)
+			(type default)
+		)
+	)
 	(bus
 		(pts
@@
 	(wire
 		(pts
+			(xy 251.46 125.73) (xy 251.46 123.19)
+		)
+		(stroke
+			(width 0)
+			(type default)
+		)
+	)
+	(wire
+		(pts
 			(xy 213.36 182.88) (xy 213.36 184.15)
 		)
@@
 	(wire
 		(pts
-			(xy 248.92 123.19) (xy 254 123.19)
+			(xy 248.92 123.19) (xy 251.46 123.19)
 		)
 		(stroke
@@
 	(global_label "ON{slash}OFF"
 		(shape input)
-		(at 251.46 123.19 270)
+		(at 251.46 125.73 270)
 		(fields_autoplaced yes)
 		(effects
@@
 		)
 		(property "Intersheetrefs" "${INTERSHEET_REFS}"
-			(at 251.46 133.6744 90)
+			(at 251.46 136.2144 90)
 			(hide yes)
 			(show_name no)
@@
 	)
 	(symbol
-		(lib_id "Device:C_Small")
-		(at 262.89 248.92 0)
-		(unit 1)
-		(body_style 1)
-		(exclude_from_sim no)
-		(in_bom yes)
-		(on_board yes)
-		(in_pos_files yes)
-		(dnp no)
-		(fields_autoplaced yes)
-		(property "Reference" "C14"
-			(at 265.43 247.6562 0)
-			(show_name no)
-			(do_not_autoplace no)
-			(effects
-				(font
-					(size 1.27 1.27)
-				)
-				(justify left)
-			)
-		)
-		(property "Value" "C_Small"
-			(at 265.43 250.1962 0)
-			(show_name no)
-			(do_not_autoplace no)
-			(effects
-				(font
-					(size 1.27 1.27)
-				)
-				(justify left)
-			)
-		)
-		(property "Footprint" "Capacitor_SMD:C_0603_1608Metric_Pad1.08x0.95mm_HandSolder"
-			(at 262.89 248.92 0)
-			(hide yes)
-			(show_name no)
-			(do_not_autoplace no)
-			(effects
-				(font
-					(size 1.27 1.27)
-				)
-			)
-		)
-		(property "Datasheet" ""
-			(at 262.89 248.92 0)
-			(hide yes)
-			(show_name no)
-			(do_not_autoplace no)
-			(effects
-				(font
-					(size 1.27 1.27)
-				)
-			)
-		)
-		(property "Description" "Unpolarized capacitor, small symbol"
-			(at 262.89 248.92 0)
-			(hide yes)
-			(show_name no)
-			(do_not_autoplace no)
-			(effects
-				(font
-					(size 1.27 1.27)
-				)
-			)
-		)
-		(pin "1"
-		)
-		(pin "2"
-		)
-		(instances
-			(project "Interface_PCB"
-				(path "/7184a9bb-5d63-4a8c-a0a1-4583480dc42d"
-					(reference "C14")
-					(unit 1)
-				)
-			)
-		)
-	)
-	(symbol
 		(lib_id "power:+5V")
 		(at 372.11 26.67 0)
@@
 	)
 	(symbol
+		(lib_id "Device:C_Small")
+		(at 262.89 248.92 0)
+		(unit 1)
+		(body_style 1)
+		(exclude_from_sim no)
+		(in_bom yes)
+		(on_board yes)
+		(in_pos_files yes)
+		(dnp no)
+		(fields_autoplaced yes)
+		(property "Reference" "C15"
+			(at 265.43 247.6562 0)
+			(show_name no)
+			(do_not_autoplace no)
+			(effects
+				(font
+					(size 1.27 1.27)
+				)
+				(justify left)
+			)
+		)
+		(property "Value" "C_Small"
+			(at 265.43 250.1962 0)
+			(show_name no)
+			(do_not_autoplace no)
+			(effects
+				(font
+					(size 1.27 1.27)
+				)
+				(justify left)
+			)
+		)
+		(property "Footprint" "Capacitor_THT:C_Radial_D10.0mm_H16.0mm_P5.00mm"
+			(at 262.89 248.92 0)
+			(hide yes)
+			(show_name no)
+			(do_not_autoplace no)
+			(effects
+				(font
+					(size 1.27 1.27)
+				)
+			)
+		)
+		(property "Datasheet" ""
+			(at 262.89 248.92 0)
+			(hide yes)
+			(show_name no)
+			(do_not_autoplace no)
+			(effects
+				(font
+					(size 1.27 1.27)
+				)
+			)
+		)
+		(property "Description" "Unpolarized capacitor, small symbol"
+			(at 262.89 248.92 0)
+			(hide yes)
+			(show_name no)
+			(do_not_autoplace no)
+			(effects
+				(font
+					(size 1.27 1.27)
+				)
+			)
+		)
+		(pin "1"
+		)
+		(pin "2"
+		)
+		(instances
+			(project "Interface_PCB"
+				(path "/7184a9bb-5d63-4a8c-a0a1-4583480dc42d"
+					(reference "C15")
+					(unit 1)
+				)
+			)
+		)
+	)
+	(symbol
 		(lib_id "1803277:1803277")
 		(at 382.27 29.21 0)
@@
 			)
 		)
-		(property "Footprint" "Capacitor_SMD:C_0603_1608Metric_Pad1.08x0.95mm_HandSolder"
+		(property "Footprint" "Capacitor_THT:C_Radial_D10.0mm_H16.0mm_P5.00mm"
 			(at 262.89 184.15 0)
 			(hide yes)
