File: ROCSAR_Hardware/Interface_PCB/_autosave-Interface_PCB.kicad_pcb (KiCad board)
At the start: 2 copper layers, 241.6 x 69.3 mm, 31 parts, among them J1 Remove Before Flight, J2 USB_A, J3 USB_A, U1 TEN 60-2422N, U2 LM2576-5.0WU, U3 LM2576-5.0WU, U4 LM2576-5.0WU, U5 LM2576-5.0WU

Commit message: Continuation of the development of the interface pcb
Parts:
- added L1: 330uH, SRR1050HA-331Y:INDPM102100X510N, F.Cu at (113.6, 63.2)
- added L2: 330uH, SRR1050HA-331Y:INDPM102100X510N, F.Cu at (113.3, 113.4)
- added L3: 330uH, SRR1050HA-331Y:INDPM102100X510N, F.Cu at (92.6, 113.4)
- added L4: 330uH, SRR1050HA-331Y:INDPM102100X510N, F.Cu at (91.6, 63.2)
- moved J2 111.8 mm to (266.5, 37.6)
- moved J3 107.5 mm to (259.6, 118.9)
- moved U3 103.5 mm to (107.2, 83.1), turned to 90 degrees
- moved C6 98.4 mm to (115.4, 70.6)
- moved U5 93.7 mm to (85.0, 32.7), turned to 90 degrees
- moved R4 87.4 mm to (110.4, 101.0)
- moved C12 83.2 mm to (93.1, 70.5), turned to 180 degrees
- moved R3 80.6 mm to (109.1, 104.8), turned to 90 degrees
- moved C4 80.6 mm to (63.4, 37.5), turned to 0 degrees
- moved R8 80.0 mm to (88.6, 50.7), turned to 0 degrees
- moved U4 79.3 mm to (86.2, 83.1), turned to 90 degrees
- moved R5 78.2 mm to (88.3, 104.8), turned to 90 degrees
- moved U2 77.5 mm to (107.4, 33.0), turned to 90 degrees
- moved C8 76.2 mm to (115.0, 120.7), turned to 180 degrees
- moved C3 75.4 mm to (63.4, 41.2), turned to 0 degrees
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Routing:
- net GND: track 71.5 -> 138.2 mm
- net +5V: track 0.00 -> 64.8 mm
- net Net-(J2-D-): track 59.3 -> 0.00 mm
- net Net-(J2-VBUS): track 53.7 -> 0.00 mm
- net Net-(J2-D+): track 51.6 -> 0.00 mm
- net Net-(U3-OUTPUT): track 0.00 -> 20.8 mm
- net Net-(U4-OUTPUT): track 0.00 -> 20.2 mm
- net Net-(U5-OUTPUT): track 8.47 -> 20.6 mm
- net Net-(U2-OUTPUT): track 8.57 -> 20.4 mm
- net +12V: track 21.8 -> 32.7 mm
- net Net-(U4-FEEDBACK): track 0.00 -> 7.74 mm
- net Net-(U3-FEEDBACK): track 0.00 -> 7.65 mm
- net (no net): track 0.00 -> 3.00 mm
- added copper zone on B.Cu, net -VDC
- added copper zone on B.Cu, net GND
Other:
- board size 241.6 x 69.3 mm -> 240 x 100 mm
